File: pcb-1.kicad_sch (KiCad schematic)
At the start: 14 parts

Commit message: Finished Schematic
Parts:
- added D1, D2, D3, D4: D_Small, Diode_SMD:D_SOD-123, symbol Device:D_Small
- added F1: 500mA, Fuse:Fuse_1206_3216Metric, symbol Device:Polyfuse_Small
- added MX1, MX2, MX3, MX4: MX-NoLED, MX_Alps_Hybrid:MX-1U, symbol MX_Alps_Hybrid:MX-NoLED
- added R4, R5: 5.1k, Resistor_SMD:R_0805_2012Metric, symbol Device:R_Small
- added U1: PRTR5V0U2X, random-keyboard-parts:SOT143B, symbol random-keyboard-parts:PRTR5V0U2X
- added USB1: HRO-TYPE-C-31-M-12, Crystal:Crystal_SMD_3225-4Pin_3.2x2.5mm, symbol Type-C:HRO-TYPE-C-31-M-12
- C1, C2, C3, C4, C5, C6, C7: renamed from C?; footprint (none) -> Capacitor_SMD:C_0805_2012Metric
- R1, R2, R3, R6: renamed from R?; footprint (none) -> Resistor_SMD:R_0805_2012Metric
- SW1: renamed from SW?; footprint (none) -> random-keyboard-parts:SKQG-1155865
- Y1: renamed from Y?; footprint (none) -> Crystal:Crystal_SMD_3225-4Pin_3.2x2.5mm
- gave numbers to parts that had none: 1
Connections:
- net +5V: now also F1.2
- net GND: now also R4.2, R5.2, U1.1 (GND), USB1.1 (GND), USB1.12 (GND), USB1.13 (SHIELD)
- net COL2: now reaches U2.10 (PB2)
- net ROW1: now reaches U2.11 (PB3)
- net ROW1: now also D3.1 (K), D4.1 (K)
- net ROW0: now reaches U2.27 (PD7)
- net ROW0: now also D1.1 (K), D2.1 (K)
- net COL1: now reaches U2.9 (PB1)
- net COL1: now also MX2.1 (COL), MX4.1 (COL)
- net D+: no longer names the net of R2.1
- net D+: now also U1.3 (IO2), USB1.5 (DN2), USB1.7 (DN1)
- net D-: no longer names the net of R3.1
- net D-: now also U1.2 (IO1), USB1.6 (DP1), USB1.8 (DP2)
- new net: D3.2 (A), MX3.2 (ROW)
- new net: R4.1, USB1.10 (CC2)
- new net: R5.1, USB1.4 (CC1)
- new net: D1.2 (A), MX1.2 (ROW)
- new net: D4.2 (A), MX4.2 (ROW)
- new net: D2.2 (A), MX2.2 (ROW)
- new net COL0: MX1.1 (COL), MX3.1 (COL)
- new net VCC: F1.1, U1.4 (VCC), USB1.11 (VBUS), USB1.2 (VBUS)
- no-connect marks 0 -> 2
Other:
- moved on the sheet: C1, C2, C3, C4, C5, C6, C7, R1, R2, R3, R6, SW1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

Commit message: PCB Preparation
Parts:
- USB1: footprint Crystal:Crystal_SMD_3225-4Pin_3.2x2.5mm -> Type-C:HRO-TYPE-C-31-M-12
Connections:
- net at R3.1, U1.2 (IO1), USB1.6 (DP1)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: now also R2.1, U1.3 (IO2), USB1.5 (DN2), USB1.7 (DN1)
Changed lines of the file:
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@@
   (junction (at 110.49 76.2) (diameter 0) (color 0 0 0 0)
   )
+  (junction (at 87.63 92.71) (diameter 0) (color 0 0 0 0)
+  )
+  (junction (at 64.77 92.71) (diameter 0) (color 0 0 0 0)
+  )
+  (junction (at 106.68 93.98) (diameter 0) (color 0 0 0 0)
+  )
   (junction (at 107.95 78.74) (diameter 0) (color 0 0 0 0)
   )
   (junction (at 66.04 104.14) (diameter 0) (color 0 0 0 0)
   )
-  (junction (at 104.14 93.98) (diameter 0) (color 0 0 0 0)
-  )
-  (junction (at 87.63 91.44) (diameter 0) (color 0 0 0 0)
-  )
   (junction (at 200.66 113.03) (diameter 0) (color 0 0 0 0)
   )
@@
   (junction (at 101.6 127) (diameter 0) (color 0 0 0 0)
   )
+  (junction (at 67.31 90.17) (diameter 0) (color 0 0 0 0)
+  )
   (junction (at 120.65 66.04) (diameter 0) (color 0 0 0 0)
   )
   (junction (at 200.66 97.79) (diameter 0) (color 0 0 0 0)
   )
-  (junction (at 67.31 91.44) (diameter 0) (color 0 0 0 0)
-  )
   (junction (at 68.58 104.14) (diameter 0) (color 0 0 0 0)
   )
@@
   (junction (at 134.62 149.86) (diameter 0) (color 0 0 0 0)
   )
-  (junction (at 64.77 93.98) (diameter 0) (color 0 0 0 0)
-  )
   (junction (at 106.68 121.92) (diameter 0) (color 0 0 0 0)
   )
   (junction (at 87.63 81.28) (diameter 0) (color 0 0 0 0)
+  )
+  (junction (at 87.63 90.17) (diameter 0) (color 0 0 0 0)
   )
   (junction (at 96.52 121.92) (diameter 0) (color 0 0 0 0)
@@
   (no_connect (at 62.23 81.28))
   (no_connect (at 62.23 96.52))
-  (wire (pts (xy 67.31 86.36) (xy 67.31 91.44))
+  (wire (pts (xy 67.31 86.36) (xy 67.31 90.17))
     (stroke (width 0) (type default) (color 0 0 0 0))
   )
@@
     (stroke (width 0) (type default) (color 0 0 0 0))
   )
+  (wire (pts (xy 87.63 90.17) (xy 106.68 90.17))
+    (stroke (width 0) (type default) (color 0 0 0 0))
+  )
   (wire (pts (xy 121.92 86.36) (xy 113.03 86.36))
     (stroke (width 0) (type default) (color 0 0 0 0))
@@
     (stroke (width 0) (type default) (color 0 0 0 0))
   )
-  (wire (pts (xy 67.31 91.44) (xy 87.63 91.44))
-    (stroke (width 0) (type default) (color 0 0 0 0))
-  )
   (wire (pts (xy 68.58 104.14) (xy 73.66 104.14))
     (stroke (width 0) (type default) (color 0 0 0 0))
@@
     (stroke (width 0) (type default) (color 0 0 0 0))
   )
+  (wire (pts (xy 87.63 92.71) (xy 114.3 92.71))
+    (stroke (width 0) (type default) (color 0 0 0 0))
+  )
   (wire (pts (xy 66.04 104.14) (xy 66.04 106.68))
     (stroke (width 0) (type default) (color 0 0 0 0))
@@
     (stroke (width 0) (type default) (color 0 0 0 0))
   )
+  (wire (pts (xy 106.68 90.17) (xy 106.68 93.98))
+    (stroke (width 0) (type default) (color 0 0 0 0))
+  )
+  (wire (pts (xy 64.77 92.71) (xy 64.77 88.9))
+    (stroke (width 0) (type default) (color 0 0 0 0))
+  )
   (wire (pts (xy 120.65 66.04) (xy 121.92 66.04))
     (stroke (width 0) (type default) (color 0 0 0 0))
   )
+  (wire (pts (xy 87.63 90.17) (xy 87.63 92.71))
+    (stroke (width 0) (type default) (color 0 0 0 0))
+  )
   (wire (pts (xy 113.03 78.74) (xy 107.95 78.74))
     (stroke (width 0) (type default) (color 0 0 0 0))
@@
     (stroke (width 0) (type default) (color 0 0 0 0))
   )
+  (wire (pts (xy 114.3 91.44) (xy 114.3 92.71))
+    (stroke (width 0) (type default) (color 0 0 0 0))
+  )
   (wire (pts (xy 106.68 127) (xy 116.84 127))
     (stroke (width 0) (type default) (color 0 0 0 0))
@@
     (stroke (width 0) (type default) (color 0 0 0 0))
   )
-  (wire (pts (xy 87.63 91.44) (xy 114.3 91.44))
+  (wire (pts (xy 64.77 92.71) (xy 87.63 92.71))
     (stroke (width 0) (type default) (color 0 0 0 0))
   )
@@
     (stroke (width 0) (type default) (color 0 0 0 0))
   )
-  (wire (pts (xy 64.77 93.98) (xy 104.14 93.98))
+  (wire (pts (xy 67.31 90.17) (xy 87.63 90.17))
     (stroke (width 0) (type default) (color 0 0 0 0))
   )
@@
     (stroke (width 0) (type default) (color 0 0 0 0))
   )
-  (wire (pts (xy 87.63 100.33) (xy 87.63 91.44))
+  (wire (pts (xy 67.31 90.17) (xy 67.31 91.44))
+    (stroke (width 0) (type default) (color 0 0 0 0))
+  )
+  (wire (pts (xy 87.63 100.33) (xy 87.63 92.71))
     (stroke (width 0) (type default) (color 0 0 0 0))
   )
@@
     (stroke (width 0) (type default) (color 0 0 0 0))
   )
-  (wire (pts (xy 64.77 93.98) (xy 64.77 88.9))
+  (wire (pts (xy 64.77 93.98) (xy 64.77 92.71))
     (stroke (width 0) (type default) (color 0 0 0 0))
   )
@@
       (effects (font (size 0.75 0.75)))
     )
-    (property "Footprint" "Crystal:Crystal_SMD_3225-4Pin_3.2x2.5mm" (id 2) (at 59.69 90.17 0)
+    (property "Footprint" "Type-C:HRO-TYPE-C-31-M-12" (id 2) (at 59.69 90.17 0)
       (effects (font (size 1.524 1.524)) hide)
     )
@@
     )
     (path "/32e04083-fbc5-4d74-977f-832005b55756"
-      (reference "USB1") (unit 1) (value "HRO-TYPE-C-31-M-12") (footprint "Crystal:Crystal_SMD_3225-4Pin_3.2x2.5mm")
+      (reference "USB1") (unit 1) (value "HRO-TYPE-C-31-M-12") (footprint "Type-C:HRO-TYPE-C-31-M-12")
     )
     (path "/f30dfd0c-ccf2-4968-9398-581e23bd1767"
